Commit message: pdz gripper (gazebo): register right_finger_joint so the <mimic> is enforced
The pdz gripper's right_finger_joint is a URDF <mimic> of left_finger_joint,
but only left_finger_joint was declared under the <ros2_control> block. The
installed gz_ros2_control 0.7.20 (Fortress build) *does* have <mimic>
emulation, but it only iterates joints registered under a <ros2_control>
block -- so the follower was left as a free, unactuated prismatic joint that
flailed under contact / inertial coupling and never closed on a part
("fingers jerk around, nothing is gripped").

Declare right_finger_joint in both lbr_one/lbr_two pdz gripper systems with a
state interface only (no command interface -- no controller drives it; the
mimic emulation writes its position each cycle). Controllers are unchanged
(still left_finger_joint only), so plan_executor_node needs no changes.
mode:=mock's GenericSystem also honours the mimic given a registered
follower, so the block is correct for mock/hardware too.

Verified: xacro expands cleanly for mode in {gazebo,mock,hardware} x
gripper=pdz and for gripper=y_gripper (no regression).

Paired with a small <dynamics damping/friction> addition on the pdz finger
joints in pdz_gripper_description/urdf/pdz_gripper_macro.xacro.

Co-Authored-By: Claude Sonnet 5 <noreply@anthropic.com>
Claude-Session: https://claude.ai/code/session_01BNtUy7WFdE6CP4jYo4diRX

File: lbr_dual_arm_description/urdf/lbr_dual_arm.xacro (robot description, xacro)
@@ -179,6 +179,13 @@
         load if used there (confirmed: "does not exist. Declared types are
         gz_ros2_control/GazeboSimSystem ign_ros2_control/IgnitionSystem", then a GUI segfault).
-        right_finger_joint is a <mimic> of left_finger_joint (see pdz_gripper_macro.xacro) so it
-        needs no interface of its own. -->
+        right_finger_joint is a mimic of left_finger_joint (see pdz_gripper_macro.xacro). It
+        carries NO command interface (no controller drives it) but it MUST still be declared
+        here with a state interface: gz_ros2_control's mimic emulation (present in the installed
+        gz_ros2_control 0.7.20 / Fortress build; it reads the URDF mimic tag and writes the
+        follower's position each update cycle, no physics constraint) only iterates joints
+        registered under a ros2_control block. Without this block the follower is left as a
+        free, unactuated prismatic joint that flails under contact / inertial coupling and
+        never closes on a part. mode:=mock's mock_components/GenericSystem also honours the
+        mimic given a registered follower, so this block is correct for both modes. -->
         <xacro:property name="pdz_gripper_hw_plugin"
             value="${'gz_ros2_control/GazeboSimSystem' if mode == 'gazebo' else 'mock_components/GenericSystem'}" />
@@ -201,4 +208,10 @@
                     <state_interface name="velocity" />
                 </joint>
+                <joint name="lbr_one_pdz_gripper_right_finger_joint">
+                    <state_interface name="position">
+                        <param name="initial_value">0.0</param>
+                    </state_interface>
+                    <state_interface name="velocity" />
+                </joint>
             </ros2_control>
             <xacro:pdz_gripper parent="lbr_two_link_ee" prefix="lbr_two_">
@@ -219,4 +232,10 @@
                     <state_interface name="velocity" />
                 </joint>
+                <joint name="lbr_two_pdz_gripper_right_finger_joint">
+                    <state_interface name="position">
+                        <param name="initial_value">0.0</param>
+                    </state_interface>
+                    <state_interface name="velocity" />
+                </joint>
             </ros2_control>
         </xacro:if>
